Commit message: rotor info added in sim and controller

File: drone_simulator/drone_description/urdf/custom_hexacopter/custom_hexacopter.xacro (robot description, xacro)
@@ -29,6 +29,6 @@
   <xacro:property name="rotor_offset_top" value="0.068" /> <!-- [m] -->
   <xacro:property name="radius_rotor" value="0.127" /> <!-- [m] -->
-  <xacro:property name="motor_constant" value="8.54858e-06" /> <!-- [kg m/s^2] -->
-  <xacro:property name="moment_constant" value="0.016" /> <!-- [m] -->
+  <xacro:property name="motor_constant" value="13.3591e-06" /> <!-- [kg m/s^2] -->
+  <xacro:property name="moment_constant" value="0.06372" /> <!-- [m] -->
   <xacro:property name="time_constant_up" value="0.0125" /> <!-- [s] -->
   <xacro:property name="time_constant_down" value="0.025" /> <!-- [s] -->

File: drone_simulator/drone_description/urdf/custom_hexacopter/custom_hexacopter_base.xacro (robot description, xacro)
@@ -20,6 +20,6 @@
   <!-- Instantiate firefly "mechanics" -->
   <xacro:include filename="$(find drone_description)/urdf/custom_hexacopter/custom_hexacopter.xacro" />
-  <!-- <xacro:include filename="$(find drone_description)/urdf/sensors/d435.xacro"
-  namespace="${namespace}" parent_link="${namespace}/base_link" /> -->
+  <xacro:include filename="$(find drone_description)/urdf/sensors/d435.xacro"
+  namespace="${namespace}" parent_link="${namespace}/base_link" />
   <!-- Instantiate a controller. -->
   <xacro:controller_plugin_macro namespace="${namespace}" imu_sub_topic="imu" />

File: drone_simulator/drone_description/urdf/sensors/d435.xacro (robot description, xacro)
@@ -41,6 +41,6 @@
         enable_visual="true">
     <box size="0.01 0.01 0.01"/>
-    <origin xyz="0.1 -0.0175 0"
-    rpy = "0 ${pi/4} 0"/>
+    <origin xyz="0.04 -0.0175 -0.06"
+    rpy = "0 ${pi/6} 0"/>
   </xacro:camera_macro>
   <xacro:camera_macro
@@ -59,6 +59,6 @@
         enable_visual="true">
     <box size="0.01 0.01 0.01"/>
-    <origin xyz="0.1 0.0325 0"
-    rpy = "0 ${pi/4} 0"/>
+    <origin xyz="0.04 0.0325 -0.06"
+    rpy = "0 ${pi/6} 0"/>
   </xacro:camera_macro>
 </robot>

Commit message: simulator - parameter updated

File: drone_simulator/drone_description/urdf/custom_hexacopter/custom_hexacopter.xacro (robot description, xacro)
@@ -16,5 +16,5 @@
   limitations under the License.
 -->
-<robot name="firefly" xmlns:xacro="http://ros.org/wiki/xacro">
+<robot name="custom_hexa" xmlns:xacro="http://ros.org/wiki/xacro">
   <!-- Properties -->
   <xacro:property name="namespace" value="$(arg namespace)" />
@@ -29,6 +29,6 @@
   <xacro:property name="rotor_offset_top" value="0.068" /> <!-- [m] -->
   <xacro:property name="radius_rotor" value="0.127" /> <!-- [m] -->
-  <xacro:property name="motor_constant" value="13.3591e-06" /> <!-- [kg m/s^2] -->
-  <xacro:property name="moment_constant" value="0.06372" /> <!-- [m] -->
+  <xacro:property name="motor_constant" value="1.336e-05" /> <!-- [kg m/s^2] -->
+  <xacro:property name="moment_constant" value="0.01569" /> <!-- [m] -->
   <xacro:property name="time_constant_up" value="0.0125" /> <!-- [s] -->
   <xacro:property name="time_constant_down" value="0.025" /> <!-- [s] -->
@@ -40,5 +40,5 @@
   <!-- Property Blocks -->
   <xacro:property name="body_inertia">
-    <inertia ixx="0.0347563" ixy="0.0" ixz="0.0" iyy="0.0458929" iyz="0.0" izz="0.0977" /> <!-- [kg m^2] [kg m^2] [kg m^2] [kg m^2] [kg m^2] [kg m^2] -->
+    <inertia ixx="0.05267" ixy="0.0" ixz="0.0" iyy="0.05290" iyz="0.0" izz="0.08524" /> <!-- [kg m^2] [kg m^2] [kg m^2] [kg m^2] [kg m^2] [kg m^2] -->
   </xacro:property>
   <!-- inertia of a single rotor, assuming it is a cuboid. Height=3mm, width=15mm -->

File: drone_simulator/drone_description/urdf/sensors/d435.xacro (robot description, xacro)
@@ -11,19 +11,4 @@
         <color rgba="0 0 0 1.0" />
     </material> -->
-  <!-- <link name="camera_link">
-    <collision>
-      <origin xyz="0 -0.0175 0" rpy="${pi/2} 0 ${pi/2}" />
-      <geometry>
-        <mesh filename="package://drone_description/meshes/sensors/d435_simple.dae" scale="1 1 1" />
-      </geometry>
-    </collision>
-    <visual>
-      <origin xyz="0 -0.0175 0" rpy="${pi/2} 0 ${pi/2}" />
-      <geometry>
-        <mesh filename="package://drone_description/meshes/sensors/d435_simple.dae" scale="1 1 1" />
-      </geometry>
-      <material name="black" />
-    </visual>
-  </link> -->
   <xacro:camera_macro
         namespace="${namespace}"
@@ -41,6 +26,6 @@
         enable_visual="true">
     <box size="0.01 0.01 0.01"/>
-    <origin xyz="0.04 -0.0175 -0.06"
-    rpy = "0 ${pi/6} 0"/>
+    <origin xyz="0.0507 -0.0175 -0.0698"
+    rpy = "0 ${pi/4} 0"/>
   </xacro:camera_macro>
   <xacro:camera_macro
@@ -59,6 +44,6 @@
         enable_visual="true">
     <box size="0.01 0.01 0.01"/>
-    <origin xyz="0.04 0.0325 -0.06"
-    rpy = "0 ${pi/6} 0"/>
+    <origin xyz="0.0507 0.0325 -0.0698"
+    rpy = "0 ${pi/4} 0"/>
   </xacro:camera_macro>
 </robot>

Commit message: Camera angle modified

File: drone_simulator/drone_description/urdf/custom_hexacopter/custom_hexacopter.xacro (robot description, xacro)
@@ -22,10 +22,10 @@
   <xacro:property name="use_mesh_file" value="true" />
   <xacro:property name="mesh_file" value="package://drone_description/meshes/custom_hexacopter/custom_hexacopter.dae" />
-  <xacro:property name="mass" value="2.9" /> <!-- [kg] -->
+  <xacro:property name="mass" value="2.790" /> <!-- [kg] -->
   <xacro:property name="body_width" value="0.80" /> <!-- [m] -->
-  <xacro:property name="body_height" value="0.53" /> <!-- [m] -->
-  <xacro:property name="mass_rotor" value="0.015" /> <!-- [kg] -->
+  <xacro:property name="body_height" value="0.625" /> <!-- [m] -->
+  <xacro:property name="mass_rotor" value="0.018333" /> <!-- [kg] -->
   <xacro:property name="arm_length" value="0.265" /> <!-- [m] -->
-  <xacro:property name="rotor_offset_top" value="0.068" /> <!-- [m] -->
+  <xacro:property name="rotor_offset_top" value="0.020" /> <!-- [m] -->
   <xacro:property name="radius_rotor" value="0.127" /> <!-- [m] -->
   <xacro:property name="motor_constant" value="1.336e-05" /> <!-- [kg m/s^2] -->

File: drone_simulator/drone_description/urdf/sensors/d435.xacro (robot description, xacro)
@@ -20,5 +20,5 @@
         image_height="480"
         image_format="L8"
-        min_distance="0.3"
+        min_distance="0.01"
         max_distance="30.0"
         noise_mean="0.0"
@@ -26,6 +26,6 @@
         enable_visual="true">
     <box size="0.01 0.01 0.01"/>
-    <origin xyz="0.0507 -0.0175 -0.0698"
-    rpy = "0 ${pi/4} 0"/>
+    <origin xyz="0.0597307 -0.0175 -0.1181178"
+    rpy = "0 ${pi/6} 0"/>
   </xacro:camera_macro>
   <xacro:camera_macro
@@ -38,5 +38,5 @@
         image_height="480"
         image_format="L8"
-        min_distance="0.3"
+        min_distance="0.01"
         max_distance="30.0"
         noise_mean="0.0"
@@ -44,6 +44,6 @@
         enable_visual="true">
     <box size="0.01 0.01 0.01"/>
-    <origin xyz="0.0507 0.0325 -0.0698"
-    rpy = "0 ${pi/4} 0"/>
+    <origin xyz="0.0597307 0.0325 -0.1181178"
+    rpy = "0 ${pi/6} 0"/>
   </xacro:camera_macro>
 </robot>

Commit message: custom hexa with d435

File: drone_simulator/drone_description/urdf/custom_hexacopter/custom_hexacopter.xacro (robot description, xacro)
@@ -22,27 +22,30 @@
   <xacro:property name="use_mesh_file" value="true" />
   <xacro:property name="mesh_file" value="package://drone_description/meshes/custom_hexacopter/custom_hexacopter.dae" />
-  <xacro:property name="mass" value="2.790" /> <!-- [kg] -->
+  <xacro:property name="mass" value="2.900" /> <!-- [kg] -->
   <xacro:property name="body_width" value="0.80" /> <!-- [m] -->
-  <xacro:property name="body_height" value="0.625" /> <!-- [m] -->
-  <xacro:property name="mass_rotor" value="0.018333" /> <!-- [kg] -->
+  <xacro:property name="body_height" value="0.54" /> <!-- [m] -->
+  <xacro:property name="mass_rotor" value="0.016" /> <!-- [kg] -->
   <xacro:property name="arm_length" value="0.265" /> <!-- [m] -->
-  <xacro:property name="rotor_offset_top" value="0.020" /> <!-- [m] -->
+  <xacro:property name="rotor_offset_top" value="0.064" /> <!-- [m] -->
   <xacro:property name="radius_rotor" value="0.127" /> <!-- [m] -->
   <xacro:property name="motor_constant" value="1.336e-05" /> <!-- [kg m/s^2] -->
   <xacro:property name="moment_constant" value="0.01569" /> <!-- [m] -->
-  <xacro:property name="time_constant_up" value="0.0125" /> <!-- [s] -->
-  <xacro:property name="time_constant_down" value="0.025" /> <!-- [s] -->
+  <xacro:property name="time_constant_up" value="0.01" /> <!-- [s] -->
+  <xacro:property name="time_constant_down" value="0.01" /> <!-- [s] -->
   <xacro:property name="max_rot_velocity" value="838" /> <!-- [rad/s] -->
   <xacro:property name="sin30" value="0.5" />
   <xacro:property name="cos30" value="0.866025403784" />
-  <xacro:property name="rotor_drag_coefficient" value="8.06428e-05" />
+  <xacro:property name="rotor_drag_coefficient" value="8.06428e-08" />
   <xacro:property name="rolling_moment_coefficient" value="0.000001" />
   <!-- Property Blocks -->
   <xacro:property name="body_inertia">
-    <inertia ixx="0.05267" ixy="0.0" ixz="0.0" iyy="0.05290" iyz="0.0" izz="0.08524" /> <!-- [kg m^2] [kg m^2] [kg m^2] [kg m^2] [kg m^2] [kg m^2] -->
+    <inertia ixx="0.05267" ixy="0" ixz="0"
+    iyy="0.05290" iyz="0"
+    izz="0.08524" />
   </xacro:property>
-  <!-- inertia of a single rotor, assuming it is a cuboid. Height=3mm, width=15mm -->
+  <!-- inertia of a single rotor, assuming it is a cuboid. width=30 mm, Height=10 mm -->
   <xacro:property name="rotor_inertia">
-    <xacro:box_inertia x="${radius_rotor}" y="0.015" z="0.003" mass="${mass_rotor*rotor_velocity_slowdown_sim}" />
+    <xacro:box_inertia x="${radius_rotor}" y="0.030" z="0.010"
+    mass="${mass_rotor}" />
   </xacro:property>
   <!-- Included URDF Files -->
@@ -54,5 +57,4 @@
     body_width="${body_width}"
     body_height="${body_height}"
-    use_mesh_file="${use_mesh_file}"
     mesh_file="${mesh_file}"
     >

File: drone_simulator/drone_description/urdf/custom_hexacopter/custom_hexacopter_base.xacro (robot description, xacro)
@@ -16,20 +16,20 @@
   limitations under the License.
 -->
-<robot name="firefly" xmlns:xacro="http://ros.org/wiki/xacro">
+<robot name="custom_hexa" xmlns:xacro="http://ros.org/wiki/xacro">
   <xacro:include filename="$(find drone_description)/urdf/component_snippets.xacro" />
-  <!-- Instantiate firefly "mechanics" -->
+  <!-- Instantiate custom hexa "mechanics" -->
   <xacro:include filename="$(find drone_description)/urdf/custom_hexacopter/custom_hexacopter.xacro" />
-  <xacro:include filename="$(find drone_description)/urdf/sensors/d435.xacro"
-  namespace="${namespace}" parent_link="${namespace}/base_link" />
+  <!-- Instantiate D435 camera sensor -->
+  <xacro:include filename="$(find drone_description)/urdf/sensors/d435_attach.urdf.xacro"
+  namespace="${namespace}"/>
   <!-- Instantiate a controller. -->
   <xacro:controller_plugin_macro namespace="${namespace}" imu_sub_topic="imu" />
-  <!-- Instantiate a ROS message interface -->
-  <!-- <xacro:ros_interface_plugin_macro namespace="${namespace}" />-->
   <xacro:if value="$(arg enable_mavlink_interface)">
     <!-- Instantiate mavlink telemetry interface. -->
     <xacro:default_mavlink_interface namespace="${namespace}" imu_sub_topic="imu" rotor_count="6" />
   </xacro:if>
-  <!-- Mount an ADIS16448 IMU. -->
-  <xacro:default_imu namespace="${namespace}" parent_link="${namespace}/base_link" />
+  <!-- Include Pixhawk 6x mini -->
+  <xacro:include filename="$(find drone_description)/urdf/sensors/px6_mini.xacro"
+  name="namespace"/>
   <xacro:if value="$(arg enable_ground_truth)">
     <xacro:ground_truth_imu_and_odometry namespace="${namespace}" parent_link="${namespace}/base_link" />

File: drone_simulator/drone_description/urdf/custom_hexacopter/multirotor_base.xacro (robot description, xacro)
@@ -19,19 +19,11 @@
   <!-- Macro for the inertia of a box -->
   <xacro:macro name="box_inertia" params="x y z mass">
-    <inertia ixx="${0.0833333 * mass * (y*y + z*z)}" ixy="0.0" ixz="0.0"
-      iyy="${0.0833333 * mass * (x*x + z*z)}" iyz="0.0"
-      izz="${0.0833333 * mass * (x*x + y*y)}" />
-  </xacro:macro>
-  <!-- Macro for the inertial properties of a box -->
-  <xacro:macro name="box_inertial" params="x y z mass *origin">
-    <inertial>
-      <mass value="${mass}" />
-      <xacro:insert_block name="origin" />
-      <xacro:box_inertia x="${x}" y="${y}" z="${z}" mass="${mass}" />
-    </inertial>
+    <inertia ixx="3.811e-7" ixy="0.0" ixz="0.0"
+      iyy="5.745e-5" iyz="0.0"
+      izz="5.719e-5" />
   </xacro:macro>
   <!-- Main multirotor link -->
   <xacro:macro name="multirotor_base_macro"
-    params="robot_namespace mass body_width body_height use_mesh_file mesh_file *inertia">
+    params="robot_namespace mass body_width body_height mesh_file *inertia">
     <link name="${robot_namespace}/base_link"></link>
     <joint name="${robot_namespace}/base_joint" type="fixed">
@@ -43,5 +35,5 @@
       <inertial>
         <mass value="${mass}" />  <!-- [kg] -->
-        <origin xyz="0 0 0" />
+        <origin xyz="0 0 0" rpy="0 0 0"/>
         <xacro:insert_block name="inertia" />
       </inertial>
@@ -72,10 +64,12 @@
   <!-- Rotor joint and link -->
   <xacro:macro name="vertical_rotor"
-    params="robot_namespace suffix direction motor_constant moment_constant parent mass_rotor radius_rotor time_constant_up time_constant_down max_rot_velocity motor_number rotor_drag_coefficient rolling_moment_coefficient color use_own_mesh mesh *origin *inertia">
+    params="robot_namespace suffix direction
+    motor_constant moment_constant parent mass_rotor
+    radius_rotor time_constant_up time_constant_down
+    max_rot_velocity motor_number rotor_drag_coefficient
+    rolling_moment_coefficient color use_own_mesh mesh *origin *inertia">
     <joint name="${robot_namespace}/rotor_${motor_number}_joint" type="continuous">
       <xacro:insert_block name="origin" />
       <axis xyz="0 0 1" />
-      <!-- TODO(ff): not currently set because it's not yet supported -->
-      <!-- <limit effort="2000" velocity="${max_rot_velocity}" /> -->
       <parent link="${parent}" />
       <child link="${robot_namespace}/rotor_${motor_number}" />

File: drone_simulator/drone_description/urdf/firefly/firefly_base.xacro (robot description, xacro)
@@ -20,6 +20,4 @@
   <!-- Instantiate firefly "mechanics" -->
   <xacro:include filename="$(find drone_description)/urdf/firefly/firefly.xacro" />
-  <xacro:include filename="$(find drone_description)/urdf/sensors/d435.xacro"
-  namespace="${namespace}" parent_link="${namespace}/base_link" />
   <!-- <xacro:include filename="$(find drone_description)/urdf/component_snippets.xacro" /> -->
   <!-- Instantiate a controller. -->

Commit message: custom hexa updated

File: drone_simulator/drone_description/urdf/custom_hexacopter/custom_hexacopter.xacro (robot description, xacro)
@@ -27,5 +27,5 @@
   <xacro:property name="mass_rotor" value="0.016" /> <!-- [kg] -->
   <xacro:property name="arm_length" value="0.265" /> <!-- [m] -->
-  <xacro:property name="rotor_offset_top" value="0.064" /> <!-- [m] -->
+  <xacro:property name="rotor_offset_top" value="0.062" /> <!-- [m] -->
   <xacro:property name="radius_rotor" value="0.127" /> <!-- [m] -->
   <xacro:property name="motor_constant" value="1.336e-05" /> <!-- [kg m/s^2] -->

File: drone_simulator/drone_description/urdf/sensors/d435_attach.urdf.xacro (robot description, xacro)
@@ -22,5 +22,5 @@
     <parent link="${namespace}/base_link"/>
     <child link="camera_mount"/>
-    <origin xyz="0.051 0 -0.088"
+    <origin xyz="0.046 0 -0.088"
     rpy="0 ${pi/6} 0"/>
   </joint>

Commit message: hexa updated

File: drone_simulator/drone_description/urdf/custom_hexacopter/custom_hexacopter.xacro (robot description, xacro)
@@ -24,5 +24,5 @@
   <xacro:property name="mass" value="2.900" /> <!-- [kg] -->
   <xacro:property name="body_width" value="0.80" /> <!-- [m] -->
-  <xacro:property name="body_height" value="0.54" /> <!-- [m] -->
+  <xacro:property name="body_height" value="0.545" /> <!-- [m] -->
   <xacro:property name="mass_rotor" value="0.016" /> <!-- [kg] -->
   <xacro:property name="arm_length" value="0.265" /> <!-- [m] -->

Commit message: simulator collision - from box to cylinder

File: drone_simulator/drone_description/urdf/custom_hexacopter/custom_hexacopter.xacro (robot description, xacro)
@@ -23,5 +23,5 @@
   <xacro:property name="mesh_file" value="package://drone_description/meshes/custom_hexacopter/custom_hexacopter.dae" />
   <xacro:property name="mass" value="2.900" /> <!-- [kg] -->
-  <xacro:property name="body_width" value="0.80" /> <!-- [m] -->
+  <xacro:property name="body_radius" value="0.40" /> <!-- [m] -->
   <xacro:property name="body_height" value="0.545" /> <!-- [m] -->
   <xacro:property name="mass_rotor" value="0.016" /> <!-- [kg] -->
@@ -55,5 +55,5 @@
     robot_namespace="${namespace}"
     mass="${mass}"
-    body_width="${body_width}"
+    body_radius="${body_radius}"
     body_height="${body_height}"
     mesh_file="${mesh_file}"

File: drone_simulator/drone_description/urdf/custom_hexacopter/multirotor_base.xacro (robot description, xacro)
@@ -25,5 +25,5 @@
   <!-- Main multirotor link -->
   <xacro:macro name="multirotor_base_macro"
-    params="robot_namespace mass body_width body_height mesh_file *inertia">
+    params="robot_namespace mass body_radius body_height mesh_file *inertia">
     <link name="${robot_namespace}/base_link"></link>
     <joint name="${robot_namespace}/base_joint" type="fixed">
@@ -49,5 +49,5 @@
         rpy="0 0 0" />
         <geometry>
-          <box size="${body_width} ${body_width} ${body_height}"/> <!-- [m] [m] [m] -->
+          <cylinder length="${body_height}" radius="${body_radius}" /> <!-- [m] -->
         </geometry>
       </collision>

Commit message: collision roll back to box from cylinder

File: drone_simulator/drone_description/urdf/custom_hexacopter/custom_hexacopter.xacro (robot description, xacro)
@@ -23,5 +23,5 @@
   <xacro:property name="mesh_file" value="package://drone_description/meshes/custom_hexacopter/custom_hexacopter.dae" />
   <xacro:property name="mass" value="2.900" /> <!-- [kg] -->
-  <xacro:property name="body_radius" value="0.40" /> <!-- [m] -->
+  <xacro:property name="body_width" value="0.80" /> <!-- [m] -->
   <xacro:property name="body_height" value="0.545" /> <!-- [m] -->
   <xacro:property name="mass_rotor" value="0.016" /> <!-- [kg] -->
@@ -55,5 +55,5 @@
     robot_namespace="${namespace}"
     mass="${mass}"
-    body_radius="${body_radius}"
+    body_width="${body_width}"
     body_height="${body_height}"
     mesh_file="${mesh_file}"

File: drone_simulator/drone_description/urdf/custom_hexacopter/custom_hexacopter_base.xacro (robot description, xacro)
@@ -21,6 +21,7 @@
   <xacro:include filename="$(find drone_description)/urdf/custom_hexacopter/custom_hexacopter.xacro" />
   <!-- Instantiate D435 camera sensor -->
-  <xacro:include filename="$(find drone_description)/urdf/sensors/d435_attach.urdf.xacro"
-  namespace="${namespace}"/>
+  <xacro:include filename="$(find drone_description)/urdf/sensors/d435_attach.urdf.xacro"/>
+  <!-- Instantiate PX6 mini IMU sensor -->
+  <xacro:include filename="$(find drone_description)/urdf/sensors/pxhawk_6x_mini.xacro"/>
   <!-- Instantiate a controller. -->
   <xacro:controller_plugin_macro namespace="${namespace}" imu_sub_topic="imu" />
@@ -29,8 +30,4 @@
     <xacro:default_mavlink_interface namespace="${namespace}" imu_sub_topic="imu" rotor_count="6" />
   </xacro:if>
-  <!-- Include Pixhawk 6x mini -->
-  <xacro:include
-  filename="$(find drone_description)/urdf/sensors/px6_mini.xacro"
-  name="namespace"/>
   <xacro:if value="$(arg enable_ground_truth)">
     <xacro:ground_truth_imu_and_odometry namespace="${namespace}" parent_link="${namespace}/base_link" />

File: drone_simulator/drone_description/urdf/custom_hexacopter/multirotor_base.xacro (robot description, xacro)
@@ -25,5 +25,5 @@
   <!-- Main multirotor link -->
   <xacro:macro name="multirotor_base_macro"
-    params="robot_namespace mass body_radius body_height mesh_file *inertia">
+    params="robot_namespace mass body_width body_height mesh_file *inertia">
     <link name="${robot_namespace}/base_link"></link>
     <joint name="${robot_namespace}/base_joint" type="fixed">
@@ -49,5 +49,5 @@
         rpy="0 0 0" />
         <geometry>
-          <cylinder length="${body_height}" radius="${body_radius}" /> <!-- [m] -->
+          <box size="${body_width} ${body_width} ${body_height}" /> <!-- [m] -->
         </geometry>
       </collision>

File: drone_simulator/drone_description/urdf/sensors/pxhawk_6x_mini.xacro (robot description, xacro)
@@ -1,19 +1,19 @@
 <?xml version="1.0"?>
-	<robot name="${namespace}" xmlns:xacro="http://ros.org/wiki/xacro">
+	<robot name="mavros" xmlns:xacro="http://ros.org/wiki/xacro">
   <!-- Mount an ADIS16448 IMU. -->
   <xacro:imu_plugin_macro
-    namespace="/mavros"
+    namespace="mavros"
     imu_suffix=""
     parent_link="${namespace}/base_link"
-    imu_topic="/mavros/imu/data_raw"
+    imu_topic="/imu/data_raw"
     mass_imu_sensor="1e-5"
     accelerometer_noise_density="0.0070708"
     accelerometer_random_walk="3.6921e-04"
-    accelerometer_bias_correlation_time="300.0"
-    accelerometer_turn_on_bias_sigma="0.0001"
+    accelerometer_bias_correlation_time="300"
+    accelerometer_turn_on_bias_sigma="0.01"
     gyroscope_noise_density="0.0004326"
     gyroscope_random_walk="1.2810e-05"
-    gyroscope_bias_correlation_time="1000.0"
-    gyroscope_turn_on_bias_sigma="0.0087"
+    gyroscope_bias_correlation_time="1000"
+    gyroscope_turn_on_bias_sigma="0.001"
   >
     <inertia ixx="1e-10" ixy="0.0" ixz="0.0"
