Commit message: sensors/d435_attach.urdf.xacro filename is modified

File: drone_simulator/drone_description/urdf/custom_hexacopter/custom_hexacopter_base.xacro (robot description, xacro)
@@ -22,4 +22,5 @@
   <!-- Instantiate D435 camera sensor -->
   <xacro:include filename="$(find drone_description)/urdf/sensors/d435_attach.urdf.xacro"/>
+  <!-- <xacro:include filename="$(find drone_description)/urdf/sensors/d435_deprecated.xacro"/> -->
   <!-- Instantiate PX6 mini IMU sensor -->
   <xacro:include filename="$(find drone_description)/urdf/sensors/pxhawk_6x_mini.xacro"/>

File: drone_simulator/drone_description/urdf/sensors/_d435.gazebo.xacro (robot description, xacro)
@@ -27,5 +27,5 @@
                                           infra_fps:=30
                                           align_depth:=false
-                                          enable_pointCloud:=true
+                                          enable_pointCloud:=false
                                           visualize:=false
                                           ">
@@ -83,5 +83,5 @@
             <type>gaussian</type>
             <mean>0.0</mean>
-            <stddev>0.05</stddev>
+            <stddev>0.001</stddev>
           </noise>
         </camera>
@@ -141,5 +141,5 @@
             <type>gaussian</type>
             <mean>0.0</mean>
-            <stddev>0.100</stddev>
+            <stddev>0.001</stddev>
           </noise>
         </camera>
@@ -157,7 +157,9 @@
       <plugin name="${topics_ns}" filename="librealsense_gazebo_plugin.so">
         <prefix>${camera_name}</prefix>
+        <noiseBase>0.003</noiseBase>
+        <noiseScale>0.005</noiseScale>
         <!-- Color camera settings -->
       	<colorUpdateRate>${color_fps}</colorUpdateRate>
-      	<colorTopicName>color/image_raw</colorTopicName>
+      	<colorTopicName>color/image_rect_raw</colorTopicName>
       	<colorOpticalframeName>${color_optical_frame}</colorOpticalframeName>
       	<colorCameraInfoTopicName>color/camera_info</colorCameraInfoTopicName>
@@ -171,11 +173,6 @@
       	<infrared2OpticalframeName>${infrared2_optical_frame}</infrared2OpticalframeName>
         <!-- Depth camera settings -->
-      	<rangeMinDepth>0.2</rangeMinDepth>
-        <xacro:unless value="${clip_distance > 0.0}">
-      	  <rangeMaxDepth>10.0</rangeMaxDepth>
-        </xacro:unless>
-        <xacro:if value="${clip_distance > 0.0}">
-          <rangeMaxDepth>${clip_distance}</rangeMaxDepth>
-        </xacro:if>
+      	<rangeMinDepth>0.175</rangeMinDepth>
+        <rangeMaxDepth>10.0</rangeMaxDepth>
         <xacro:unless value="${align_depth}">
         	<depthUpdateRate>${depth_fps}</depthUpdateRate>

File: drone_simulator/drone_description/urdf/sensors/_d435.urdf.xacro (robot description, xacro)
@@ -18,12 +18,12 @@
                                           enable_pointCloud:=false
                                           clip_distance:=-1.0
-                                          depth_width:=1280
-                                          depth_height:=720
+                                          depth_width:=640
+                                          depth_height:=480
                                           depth_fps:=30
                                           infra_width:=640
                                           infra_height:=480
                                           infra_fps:=30
-                                          color_width:=1920
-                                          color_height:=1080
+                                          color_width:=640
+                                          color_height:=480
                                           color_fps:=30
                                           visualize:=false

File: drone_simulator/drone_description/urdf/sensors/d435_attach.urdf.xacro (robot description, xacro)
@@ -26,5 +26,5 @@
   </joint>
   <!-- d435  frame definition can be found at https://github.com/IntelRealSense/librealsense/blob/master/doc/d435i.md -->
-  <xacro:include filename="$(find realsense_gazebo_description)/urdf/_d435.urdf.xacro"/>
+  <xacro:include filename="$(find drone_description)/urdf/sensors/_d435.urdf.xacro"/>
   <xacro:sensor_d435  parent="camera_mount" name="camera" topics_ns="camera" visualize="true">
     <origin xyz="0 0 0" rpy="0.0 0.0 0.0"/>

File: drone_simulator/drone_description/urdf/sensors/d435_deprecated.xacro (robot description, xacro)
@@ -31,5 +31,5 @@
     <visual>
       <geometry>
-        <mesh filename="package://drone_description/meshes/sensors/d435_modified.dae"
+        <mesh filename="package://drone_description/meshes/sensors/d435.dae"
         scale = "1 1 1"/>
       </geometry>
@@ -171,5 +171,5 @@
     <child link="camera_link"/>
     <origin xyz="0 0 0"
-    rpy="${-pi/2} 0 ${-pi/2}"/>
+    rpy="0 0 0"/>
   </joint>
   <joint name="camera_depth_frame_joint" type="fixed">
@@ -181,5 +181,5 @@
     <parent link="camera_depth_frame"/>
     <child link="camera_depth_optical_frame"/>
-    <origin xyz="0 0 0" rpy="${pi/2} ${-pi/2} 0"/>
+    <origin xyz="0 0 0" rpy="${-pi/2} 0 ${-pi/2}"/>
   </joint>
   <joint name="camera_infra1_frame_joint" type="fixed">
@@ -294,5 +294,5 @@
         <baseline>0.01</baseline>
         <updateRate>30.0</updateRate>
-        <cameraName>camera</cameraName>
+        <cameraName></cameraName>
         <horizontal_fov>1.5708</horizontal_fov>
         <depthNoiseModelName>D435</depthNoiseModelName>

Commit message: Modify imu model again by multiplicatin or dividing sqrt(t)

File: drone_simulator/drone_description/urdf/custom_hexacopter/custom_hexacopter_base.xacro (robot description, xacro)
@@ -23,6 +23,5 @@
   <xacro:include filename="$(find drone_description)/urdf/sensors/d435_attach.urdf.xacro"/>
   <!-- Instantiate PX6 mini IMU sensor -->
-  <!-- <xacro:include filename="$(find drone_description)/urdf/sensors/pxhawk_6x_mini.xacro"/> -->
-    <xacro:include filename="$(find drone_description)/urdf/sensors/pxhawk_6x_mini_v2.xacro"/>
+    <xacro:include filename="$(find drone_description)/urdf/sensors/pxhawk_6x_mini.xacro"/>
   <!-- Instantiate a controller. -->
   <xacro:controller_plugin_macro namespace="${namespace}" imu_sub_topic="imu" />

File: drone_simulator/drone_description/urdf/sensors/pxhawk_6x_mini.xacro (robot description, xacro)
@@ -1,6 +1,50 @@
 <?xml version="1.0"?>
 	<robot name="mavros" xmlns:xacro="http://ros.org/wiki/xacro">
-  <!-- Mount an Pixhawk 6x mini. -->
-  <xacro:imu_plugin_macro
+	<xacro:macro name="px4_6x_mini_macro"
+	 params="namespace
+	 	imu_suffix
+		parent_link
+		imu_topic
+		mass_imu_sensor
+		gyroscope_noise_density
+		gyroscope_random_walk
+    gyroscope_full_scale
+		accelerometer_noise_density
+		accelerometer_random_walk
+    accelerometer_full_scale
+		*inertia
+		*origin">
+		<!-- IMU link -->
+    <link name="${namespace}/imu${imu_suffix}_link">
+      <inertial>
+        <xacro:insert_block name="inertia" />
+        <mass value="${mass_imu_sensor}" />  <!-- [kg] -->
+        <origin xyz="0 0 0" rpy="0 0 0" />
+      </inertial>
+    </link>
+		<!-- IMU joint -->
+    <joint name="${namespace}/imu${imu_suffix}_joint" type="revolute">
+      <xacro:insert_block name="origin" />
+      <parent link="${parent_link}" />
+      <child link="${namespace}/imu${imu_suffix}_link" />
+      <limit upper="0" lower="0" effort="0" velocity="0" />
+    </joint>
+    <gazebo>
+      <plugin filename="libdrone_gazebo_imu_plugin.so" name="libdrone_gazebo_imu${imu_suffix}_plugin">
+      <!-- A good description of the IMU parameters can be found in the kalibr documentation:
+           https://github.com/ethz-asl/kalibr/wiki/IMU-Noise-Model-and-Intrinsics -->
+        <robotNamespace>${namespace}</robotNamespace> <!-- (string, required): ros namespace in which the messages are published -->
+        <linkName>${namespace}/imu${imu_suffix}_link</linkName> <!-- (string, required): name of the body which holds the IMU sensor -->
+        <imuTopic>${imu_topic}</imuTopic> <!-- (string): name of the sensor output topic and prefix of service names (defaults to imu) -->
+        <gyroNoiseDensity>${gyroscope_noise_density}</gyroNoiseDensity> <!-- Gyroscope noise density (two-sided spectrum) [rad/s/sqrt(Hz)] -->
+        <gyroRandomWalk>${gyroscope_random_walk}</gyroRandomWalk> <!-- Gyroscope bias random walk [rad/s/s/sqrt(Hz)] -->
+        <accNoiseDensity>${accelerometer_noise_density}</accNoiseDensity> <!-- Accelerometer noise density (two-sided spectrum) [m/s^2/sqrt(Hz)] -->
+        <accRandomWalk>${accelerometer_random_walk}</accRandomWalk> <!-- Accelerometer bias random walk. [m/s^2/s/sqrt(Hz)] -->
+        <accFullScale>${accelerometer_full_scale}</accFullScale> <!-- Accelerometer full scale range [m/s^2] -->
+        <gyroFullScale>${gyroscope_full_scale}</gyroFullScale> <!-- Gyroscope full scale range [deg/s] -->
+      </plugin>
+    </gazebo>
+  </xacro:macro>
+  <xacro:px4_6x_mini_macro
     namespace="mavros"
     imu_suffix=""
@@ -10,11 +54,8 @@
     accelerometer_noise_density="0.0070708"
     accelerometer_random_walk="3.6921e-04"
-    accelerometer_bias_correlation_time="300"
-    accelerometer_turn_on_bias_sigma="1e-6"
+    accelerometer_full_scale="32.0"
     gyroscope_noise_density="0.0004326"
     gyroscope_random_walk="1.2810e-05"
-    gyroscope_bias_correlation_time="1000"
-    gyroscope_turn_on_bias_sigma="1e-6"
-  >
+    gyroscope_full_scale="4000.0">
     <inertia ixx="1e-10" ixy="0.0" ixz="0.0"
              iyy="1e-10" iyz="0.0"
@@ -22,4 +63,4 @@
     <origin xyz="0.0 0.0 0.03873"
             rpy="0.0 0.0 0.0" />
-  </xacro:imu_plugin_macro>
+  </xacro:px4_6x_mini_macro>
 </robot>
