Commit message: cmd converter included

File: drone_simulator/drone_description/urdf/custom_hexacopter/multirotor_base.xacro (robot description, xacro)
@@ -35,5 +35,5 @@
       <inertial>
         <mass value="${mass}" />  <!-- [kg] -->
-        <origin xyz="0 0 0" rpy="0 0 0"/>
+        <origin xyz="0.01 0 0" rpy="0 0 0"/>
         <xacro:insert_block name="inertia" />
       </inertial>

File: drone_simulator/drone_description/urdf/sensors/pxhawk_6x_mini.xacro (robot description, xacro)
@@ -47,14 +47,14 @@
   </xacro:macro>
   <xacro:px4_6x_mini_macro
-    namespace="mavros"
+    namespace="mavros_sim"
     imu_suffix=""
     parent_link="${namespace}/base_link"
     imu_topic="/imu/data_raw"
     mass_imu_sensor="1e-5"
-    accelerometer_noise_density="0.004997776"
-    accelerometer_random_walk="3.6921e-05"
+    accelerometer_noise_density="9.995552e-4"
+    accelerometer_random_walk="3.6921e-07"
     accelerometer_full_scale="32.0"
-    gyroscope_noise_density="0.0003059355"
-    gyroscope_random_walk="1.2810e-06"
+    gyroscope_noise_density="6.01207e-05"
+    gyroscope_random_walk="3.059355e-05"
     gyroscope_full_scale="4000.0">
     <inertia ixx="1e-10" ixy="0.0" ixz="0.0"

Commit message: rosparam updated

File: drone_simulator/drone_description/urdf/custom_hexacopter/multirotor_base.xacro (robot description, xacro)
@@ -35,5 +35,5 @@
       <inertial>
         <mass value="${mass}" />  <!-- [kg] -->
-        <origin xyz="0.01 0 0" rpy="0 0 0"/>
+        <origin xyz="0.02 0.03 0" rpy="0 0 0"/>
         <xacro:insert_block name="inertia" />
       </inertial>

Commit message: updated control gain and ekf

File: drone_simulator/drone_description/urdf/custom_hexacopter/multirotor_base.xacro (robot description, xacro)
@@ -49,5 +49,6 @@
         rpy="0 0 0" />
         <geometry>
-          <box size="${body_width} ${body_width} ${body_height}" /> <!-- [m] -->
+          <box size="${body_width} ${body_width} ${body_height}" /> [m]
+          <!-- <mesh filename="${mesh_file}" scale="1 1 1" /> -->
         </geometry>
       </collision>
