Commit message: parameter updated

File: drone_simulator/drone_description/urdf/sensors/_d435.urdf.xacro (robot description, xacro)
@@ -29,5 +29,5 @@
                                           visualize:=false
                                           *origin">
-    <xacro:property name="M_PI" value="3.1415926535897931"/>
+    <xacro:property name="M_PI" value="3.14159265358979323846"/>
     <!-- The following values are approximate, and the camera node
      publishing TF values with actual calibrated camera extrinsic values -->

File: drone_simulator/drone_description/urdf/sensors/d435_attach.urdf.xacro (robot description, xacro)
@@ -1,4 +1,5 @@
 <?xml version="1.0"?>
 <robot name="realsense_cameras" xmlns:xacro="http://ros.org/wiki/xacro">
+  <xacro:property name="pi" value="3.14159265358979323846"/>
   <link name="camera_mount">
     <visual>
@@ -23,5 +24,5 @@
     <child link="camera_mount"/>
     <origin xyz="0.046 0 -0.088"
-    rpy="0 ${pi/6} 0"/>
+    rpy="0 ${pi/6.0} 0"/>
   </joint>
   <!-- d435  frame definition can be found at https://github.com/IntelRealSense/librealsense/blob/master/doc/d435i.md -->

File: drone_simulator/drone_description/urdf/sensors/pxhawk_6x_mini.xacro (robot description, xacro)
@@ -52,9 +52,9 @@
     imu_topic="/imu/data_raw"
     mass_imu_sensor="1e-5"
-    accelerometer_noise_density="0.00658978579"
-    accelerometer_random_walk="0.0006166810650256017"
+    accelerometer_noise_density="0.004997776"
+    accelerometer_random_walk="3.6921e-04"
     accelerometer_full_scale="32.0"
-    gyroscope_noise_density="0.00037331694"
-    gyroscope_random_walk="1.808187069983041e-05"
+    gyroscope_noise_density="0.0003059355"
+    gyroscope_random_walk="1.2810e-05"
     gyroscope_full_scale="4000.0">
     <inertia ixx="1e-10" ixy="0.0" ixz="0.0"
